File: badge/hardware/board/DC24-Darknet_Badge-shield.sch (EAGLE design)
At the start: 54 parts, among them Q1 SOP22, SW0 SWITCH_TACTILETACTILE-2PIN-NA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, SW1 SWITCH_TACTILETACTILE-2PIN-NA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, SW2 SWITCH_TACTILETACTILE-2PIN-NA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, SW3 SWITCH_TACTILETACTILE-2PIN-NA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, SW4 SWITCH_TACTILETACTILE-2PIN-NA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, SW5 SWITCH_TACTILETACTILE-2PIN-NA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, SW6 SWITCH_TACTILETACTILE-2PIN-NA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, SW7 SWITCH_TACTILETACTILE-2PIN-NA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, SW8 SWITCH_TACTILETACTILE-2PIN-NA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

Commit message: moved board files over so we don't lose them
Parts:
- removed D1: VT1045CTO262-H, SYNShop:VT1045CTO262-H
- removed LED10: IR, SYNShop:LEDLED5MM_EDGE
- removed LED11: STATUS, SYNShop:LEDLED5MM_EDGE
- removed Q1: SOP22, SYNShop:SOP22
- removed R2, R3: 10K, SYNShop:RESISTORAXIAL-0.3
- removed R4, R5: 56, SYNShop:RESISTORAXIAL-0.3
- removed RESET: SWITCH_TACTILETACTILE-2PIN-NARROW, SYNShop:SWITCH_TACTILETACTILE-2PIN-NARROW
- removed U$14, U$17: HEADER_11PIN, SYNShop:HEADER_11PIN
- removed U$15: STM32_DEV_BOARDSTM32_DEV_BOARD, SYNShop:STM32_DEV_BOARDSTM32_DEV_BOARD
- removed U$22: DN_LOGO, SYNShop:DN_LOGO
- removed U$3, U$4, U$5: AAA_BATTERYAAA_BATTERY_CLIP, SYNShop:AAA_BATTERYAAA_BATTERY_CLIP
Connections:
- removed net A0: U$15.A0
- removed net B8: U$15.B8
- removed net C13: U$15.C13
- removed net C14: U$15.C14
- removed net C15: U$15.C15
- removed net FTDI_UART3_RX: U$15.B11
- removed net FTDI_UART3_TX: U$15.B10
- removed net IR_LED_STATUS: R5.1, U$15.B1
- removed net IR_TIM2_CH2: LED10.C, U$15.A1
- removed net IR_UART2_RX: Q1.OUT, U$15.A3
- removed net IR_UART2_TX: R4.1, U$15.A2
- removed net N$1: LED10.A, R4.2
- removed net N$13: U$3.-V, U$4.+V
- removed net N$14: U$4.-V, U$5.+V
- removed net N$2: LED11.A, R5.2
- removed net N$3: D1.PIN1, D1.PIN3, U$3.+V
- removed net RESET: RESET.A, U$15.RST
- removed net USB_DM: U$15.A11
- removed net USB_DP: U$15.A12
- net 3.3V: no longer Q1.VS, R2.2, R3.2, U$15.3.3V, U$15.3.3V2, U$15.VB, U$17.P$10
- net 5V: no longer D1.PIN2, U$15.5V, U$17.P$1
- net GND: no longer LED11.C, Q1.GND, RESET.C, U$15.GND1, U$15.GND2, U$15.GND3, U$17.P$11, U$5.-V
- net KEYBOARD_X1: no longer U$14.P$1, U$15.B12
- net KEYBOARD_X2: no longer U$14.P$2, U$15.B13
- net KEYBOARD_X3: no longer U$14.P$3, U$15.B14
- net KEYBOARD_X4: no longer U$14.P$4, U$15.B15
- net KEYBOARD_Y1: no longer U$14.P$5, U$15.A8
- net KEYBOARD_Y2: no longer U$14.P$6, U$15.A9
- net KEYBOARD_Y3: no longer U$14.P$7, U$15.A10
- net LED_OUT1: no longer U$14.P$8, U$15.A15
- net LED_OUT2: no longer U$14.P$9, U$15.B3
- net LED_OUT3: no longer U$14.P$10, U$15.B4
- net LED_OUT4: no longer U$14.P$11, U$15.B5
- net OLED_I2C1_SCL: no longer R2.1, U$15.B6, U$17.P$2
- net OLED_I2C1_SDA: no longer R3.1, U$15.B7, U$17.P$3
- net RFM69_INTERRUPT_DIO0: no longer U$15.B0, U$17.P$4
- net RFM69_RESET: no longer U$15.B9, U$17.P$9
- net RFM69_SPI_MISO: no longer U$15.A6, U$17.P$5
- net RFM69_SPI_MOSI: no longer U$15.A7, U$17.P$6
- net RFM69_SPI_NSS: no longer U$15.A4, U$17.P$8
- net RFM69_SPI_SCK: no longer U$15.A5, U$17.P$7
